File: mm_motor.kicad_sch (KiCad schematic)
At the start: 1 part, among them M1 N20_encoder

Commit message: tp2
Parts:
- added C11: 0.1uF, Capacitor_SMD:C_0603_1608Metric, symbol Device:C
- added C12: 2.2uF, Capacitor_SMD:C_0603_1608Metric, symbol Device:C
- added J3: Conn_01x06_Pin, Connector_PinHeader_2.54mm:PinHeader_1x06_P2.54mm_Vertical, symbol Connector:Conn_01x06_Pin
Connections:
- net C1: now also J3.3 (Pin_3)
- net C2: now also J3.4 (Pin_4)
- net MA: now also J3.1 (Pin_1)
- net MB: now also J3.6 (Pin_6)
- new net +BATT: C11.1, C12.1, J3.5 (Pin_5)
- new net GND: C11.2, C12.2, J3.2 (Pin_2)
Other:
- moved on the sheet: M1

Commit message: 31/01
Parts:
- removed C11: 0.1uF, Capacitor_SMD:C_0603_1608Metric, symbol Device:C
- added R19, R21: 100, Resistor_SMD:R_0603_1608Metric, symbol Device:R
- renumbered C12 to C13
Connections:
- net C1: now also R19.1; no longer J3.3 (Pin_3)
- net C2: now also R21.1; no longer J3.4 (Pin_4)
- new net: J3.4 (Pin_4), R21.2
- new net: J3.3 (Pin_3), R19.2
Other:
- moved on the sheet: C13
