File: mm_motor_control.kicad_sch (KiCad schematic)
At the start: 0 parts

Commit message: tp2
Parts:
- added C10: 2.2uF, Capacitor_SMD:C_0603_1608Metric, symbol Device:C
- added C14: 22nF, Capacitor_SMD:C_0603_1608Metric, symbol Device:C
- added C15: 0.1uF, Capacitor_SMD:C_0603_1608Metric, symbol Device:C_Polarized
- added R10: 100K, Resistor_SMD:R_0603_1608Metric, symbol Device:R
- added R11: 100k, Resistor_SMD:R_0603_1608Metric, symbol Device:R
- added R13, R14, R15, R16, R17: 100, Resistor_SMD:R_0603_1608Metric, symbol Device:R
- added R20: 1K, Resistor_SMD:R_0603_1608Metric, symbol Device:R
- added R21: 47K, Resistor_SMD:R_0603_1608Metric, symbol Device:R
- added R22, R23: 330m, Resistor_SMD:R_0603_1608Metric, symbol Device:R
- added U5: STSPIN240, Package_DFN_QFN:VQFN-16-1EP_3x3mm_P0.5mm_EP1.8x1.8mm, symbol Driver_Motor:STSPIN240
Connections:
- net EN: now also R13.2, U5.13 (EN/FLT)
- net FAULT: now also R13.1
- net OUT_A1: now also R14.2
- net OUT_A2: now also R15.2
- net OUT_B1: now also R16.2
- net OUT_B2: now also R17.2
- net PHASE_A: now also U5.1 (PHA)
- net PHASE_B: now also U5.15 (PHB)
- net PWM_A: now also U5.2 (PWMA)
- net PWM_B: now also U5.16 (PWMB)
- net STBY/RESET: now also U5.14 (STBY/RESET)
- new net: R15.1, U5.5 (OUTA2)
- new net: R20.1, R21.1, U5.12 (TOFF)
- new net: C14.1, R20.2
- new net: R22.1, U5.4 (SENSEA)
- new net: R17.1, U5.8 (OUTB2)
- new net: R10.2, R11.1, U5.11 (REF)
- new net: R14.1, U5.3 (OUTA1)
- new net: R16.1, U5.10 (OUTB1)
- new net: R23.1, U5.9 (SENSEB)
- new net +BATT: C10.1, C15.1, R10.1, U5.6 (VS)
- new net GND: C10.2, C14.2, C15.2, R11.2, R21.2, R22.2, R23.2, U5.17 (EPAD), U5.7 (GND)

Commit message: 31/01
Parts:
- removed C15: 0.1uF, Capacitor_SMD:C_0603_1608Metric, symbol Device:C_Polarized
- removed R14, R15, R16, R17: 100, Resistor_SMD:R_0603_1608Metric, symbol Device:R
- added C11: 1nF, Capacitor_SMD:C_0603_1608Metric, symbol Device:C
- R13: renamed from R10; value 100K -> 10k
- R14: renamed from R11; value 100k -> 10k
- R17: renamed from R13; value 100 -> 10k
- renumbered C14 to C10, C10 to C12, R23 to R11, R22 to R12, R20 to R15, R21 to R16, U5 to U3
Connections:
- net EN: now also R17.1; no longer R17.2, U3.13 (EN/FLT)
- net FAULT: now also R17.2, U3.13 (EN/FLT), C11.1; no longer R17.1
- net GND: now also C11.2
- net OUT_A1: now also U3.3 (OUTA1)
- net OUT_A2: now also U3.5 (OUTA2)
- net OUT_B1: now also U3.10 (OUTB1)
- net OUT_B2: now also U3.8 (OUTB2)
Other:
- moved on the sheet: C12, R13, R14, R17
