File: minimouse.kicad_pcb (KiCad board)
At the start: 2 copper layers, 90 x 85 mm, 22 parts, among them J1 Conn_ARM_JTAG_SWD_10, J5 Conn_01x02, M1 N20_encoder, M2 N20_encoder, U1 STM32F030C8Tx, U4 HC-SR04

Commit message: 31/01
Parts:
- removed R7: 100, Resistor_SMD:R_0603_1608Metric
- added C10: 22nF, Capacitor_SMD:C_0603_1608Metric, F.Cu at (159.7, 98.3)
- added C11: 1nF, Capacitor_SMD:C_0603_1608Metric, F.Cu at (154.6, 96.0)
- added C12: 2.2uF, Capacitor_SMD:C_0603_1608Metric, F.Cu at (149.8, 104.5)
- added C13: 2.2uF, Capacitor_SMD:C_0603_1608Metric, F.Cu at (172.9, 100.2)
- added C14: 2.2uF, Capacitor_SMD:C_0603_1608Metric, F.Cu at (133.7, 100.4)
- added C15: 2.2uF, Capacitor_SMD:C_0603_1608Metric, F.Cu at (155.7, 71.1)
- added C7: 2.2uF, Capacitor_SMD:C_0603_1608Metric, F.Cu at (168.4, 74.9)
- added C8: 1pF, Capacitor_SMD:C_0603_1608Metric, F.Cu at (172.0, 78.0)
- added C9: 1pF, Capacitor_SMD:C_0603_1608Metric, F.Cu at (173.6, 72.2)
- added D1: red_LED_1.7V_20mA, LED_SMD:LED_0603_1608Metric, F.Cu at (176.1, 76.2)
- added J2: Conn_01x04_Pin, Connector_PinHeader_2.54mm:PinHeader_1x04_P2.54mm_Vertical, F.Cu at (164.4, 73.1)
- added J3: Conn_01x06_Pin, Connector_PinHeader_2.54mm:PinHeader_1x06_P2.54mm_Vertical, F.Cu at (162.8, 103.8)
- added J4: Conn_01x06_Pin, Connector_PinHeader_2.54mm:PinHeader_1x06_P2.54mm_Vertical, F.Cu at (123.6, 103.8)
- added R10: 100, Resistor_SMD:R_0603_1608Metric, F.Cu at (152.4, 78.4)
- added R11: 330m, Resistor_SMD:R_0603_1608Metric, F.Cu at (154.6, 104.0)
- added R12: 330m, Resistor_SMD:R_0603_1608Metric, F.Cu at (141.3, 100.5)
- added R13: 10k, Resistor_SMD:R_0603_1608Metric, F.Cu at (154.6, 100.6)
- added R14: 10k, Resistor_SMD:R_0603_1608Metric, F.Cu at (154.6, 102.1)
- added R15: 1K, Resistor_SMD:R_0603_1608Metric, F.Cu at (154.6, 97.5)
- added R16: 47K, Resistor_SMD:R_0603_1608Metric, F.Cu at (154.6, 99.0)
- added R17: 10k, Resistor_SMD:R_0603_1608Metric, F.Cu at (153.0, 94.4)
- added R18: 80, Resistor_SMD:R_0603_1608Metric, F.Cu at (176.1, 73.0)
- added R19: 100, Resistor_SMD:R_0603_1608Metric, F.Cu at (167.9, 100.3)
- added R20: 100, Resistor_SMD:R_0603_1608Metric, F.Cu at (128.7, 100.4)
- added R21: 100, Resistor_SMD:R_0603_1608Metric, F.Cu at (170.4, 100.3)
- added R22: 100, Resistor_SMD:R_0603_1608Metric, F.Cu at (131.2, 100.4)
- added R23: 100, Resistor_SMD:R_0603_1608Metric, F.Cu at (151.3, 71.9)
- added U2: LP5907MFX-3.3, Package_TO_SOT_SMD:SOT-23-5, F.Cu at (173.2, 74.7)
- added U3: STSPIN240, Package_DFN_QFN:VQFN-16-1EP_3x3mm_P0.5mm_EP1.8x1.8mm, F.Cu at (149.2, 99.2)
- moved C5 36.4 mm to (160.7, 91.5), turned to -90 degrees
- moved C2 20.6 mm to (163.8, 91.5), turned to -90 degrees
- moved C3 20.2 mm to (162.2, 91.5), turned to -90 degrees
- moved C6 16.5 mm to (157.6, 91.5), turned to -90 degrees
- moved C1 13.9 mm to (146.3, 77.0), turned to 90 degrees
- moved R1 6.95 mm to (152.4, 74.7), turned to 0 degrees
- moved J1 5.52 mm to (158.4, 83.7)
- moved R5 5.05 mm to (148.2, 94.9)
- moved R4 5.03 mm to (146.7, 94.9)
- moved R6 4.58 mm to (150.7, 94.9)
- moved C4 4.31 mm to (159.1, 91.5), turned to -90 degrees
- moved R3 4.25 mm to (145.2, 95.8)
- moved R9 4.18 mm to (148.1, 77.0)
- moved U1 2.80 mm to (150.3, 86.8)
- moved BOOT0 1.85 mm to (155.7, 76.9), turned to -90 degrees
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Connections:
- R8 pad 1: /mcu/UART1_TX -> /external_uart/EXT_UART_RX
- U1 pad 19: Net-(U1-PB1) -> /mcu/OUT_B1
- U1 pad 43: /mcu/UART1_RX -> /external_uart/EXT_UART_TX
- U4 pad 4: +3V3 -> +3.3V
Routing:
- net GND: track 0.00 -> 368.4 mm, vias 0 -> 1
- net +BATT: track 0.00 -> 186.9 mm, vias 0 -> 1
- net +3.3V: track 0.00 -> 125.9 mm
- net /motorA/MB: track 0.00 -> 30.9 mm
- net /motorB/MA: track 0.00 -> 29.4 mm
- net /mcu/TIM3_CH2: track 0.00 -> 25.8 mm, vias 0 -> 2
- net /mcu/TIM3_CH1: track 0.00 -> 24.7 mm, vias 0 -> 2
- net /mcu/~{RESET}: track 0.00 -> 24.5 mm, vias 0 -> 2
- net /mcu/TIM2_CH1: track 0.00 -> 24.1 mm
- net /mcu/TIM2_CH2: track 0.00 -> 22.5 mm
- net /mcu/SWO: track 0.00 -> 17.4 mm
- net /mcu/BOOT0: track 0.00 -> 15.2 mm
- net /motorA/MA: track 0.00 -> 14.9 mm
- net /mcu/SWDCLK: track 0.00 -> 14.6 mm
- net /motorB/MB: track 0.00 -> 14.3 mm
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- added copper zone on B.Cu, net GND

Commit message: 05/02
Parts:
- added 3.3V1: TestPoint, TestPoint:TestPoint_Pad_D1.5mm, F.Cu at (144.5, 80.0)
- added BATT1: TestPoint, TestPoint:TestPoint_Pad_D1.5mm, F.Cu at (168.2, 80.9)
- added C16: 100nF, Capacitor_SMD:C_0603_1608Metric, F.Cu at (173.5, 88.4)
- added D2: BZT52Bxx, Diode_SMD:D_SOD-123F, F.Cu at (121.0, 91.0)
- added D3: red_LED_1.7V_20mA, LED_SMD:LED_0603_1608Metric, F.Cu at (154.5, 76.9)
- added GND1: TestPoint, TestPoint:TestPoint_Pad_D1.5mm, F.Cu at (165.0, 99.0)
- added Q1: DMP3013SFV, Package_SON:Diodes_PowerDI3333-8, F.Cu at (120.6, 96.1)
- added R24: 10K, Resistor_SMD:R_0603_1608Metric, F.Cu at (171.2, 80.9)
- added R25: 10K, Resistor_SMD:R_0603_1608Metric, F.Cu at (144.5, 77.1)
- added R26: 85, Resistor_SMD:R_0603_1608Metric, F.Cu at (151.4, 76.9)
- added R7: 100K, Resistor_SMD:R_0603_1608Metric, F.Cu at (120.5, 87.7)
- added SW1: SW_Push, Button_Switch_SMD:Panasonic_EVQPUK_EVQPUB, F.Cu at (168.9, 88.3)
- moved R22 4.36 mm to (135.5, 100.4)
- moved C14 4.35 mm to (138.1, 100.4)
- moved J4 4.34 mm to (127.9, 103.8)
- moved R20 4.32 mm to (133.0, 100.4)
- moved BOOT0 3.15 mm to (158.9, 76.9)
- moved R12 1.98 mm to (143.3, 100.5)
- moved R17 0.48 mm to (153.1, 94.0)
Connections:
- C15 pad 1: +3.3V -> +BATT
- J5 pad 2: +BATT -> Net-(J5-Pin_2)
- U4 pad 4: +3.3V -> +BATT
Routing:
- net GND: track 368.4 -> 243.3 mm, vias 1 -> 3
- net /mcu/~{RESET}: track 24.5 -> 94.1 mm
- net Net-(J5-Pin_2): track 0.00 -> 50.2 mm
- net +3.3V: track 125.9 -> 94.5 mm, vias 0 -> 2
- net +BATT: track 186.9 -> 198.5 mm, vias 1 -> 2
- net Net-(D2-A): track 0.00 -> 7.00 mm
- net /motorB/MA: track 29.4 -> 22.7 mm
- net /mcu/TIM2_CH2: track 22.5 -> 16.2 mm
- net /mcu/TIM2_CH1: track 24.1 -> 18.3 mm
- net /motorB/MB: track 14.3 -> 9.95 mm
- net /mcu/BOOT0: track 15.2 -> 17.9 mm
- net /external_uart/EXT_UART_TX: track 5.47 -> 7.61 mm
- net Net-(U3-SENSEA): track 7.01 -> 5.01 mm
- net Net-(D3-A): track 0.00 -> 1.44 mm
- net /mcu/TIM15_CH1: track 7.30 -> 6.69 mm
Other:
- board text added: "+"
- board text added: "-"
- board text added: "3.3V"
- board text added: "BATT"
- board text added: "C1"
- board text added: "C2"
- board text added: "ECHO"
- board text added: "EXT"
- board text added: "GND"
- board text added: "MA"
- board text added: "MB"
- board text added: "NET"
- board text added: "OUT"
- board text added: "RESET"
- board text added: "SWDCLK"
- board text added: "SWDIO"
- board text added: "SWO"
