File: mm_mcu.kicad_sch (KiCad schematic)
At the start: 17 parts, among them J1 Conn_ARM_JTAG_SWD_10, U1 STM32F030C8Tx

Commit message: 05/02
Parts:
- added C16: 100nF, Capacitor_SMD:C_0603_1608Metric, symbol Device:C
- added D3: red_LED_1.7V_20mA, LED_SMD:LED_0603_1608Metric, symbol Device:LED
- added R26: 85, Resistor_SMD:R_0603_1608Metric, symbol Device:R
- added SW1: SW_Push, Button_Switch_SMD:Panasonic_EVQPUK_EVQPUB, symbol Switch:SW_Push
Connections:
- net GND: now also C16.2, D3.1 (K), SW1.1
- net UART1_RX: now also R26.2
- net ~{RESET}: now also C16.1, SW1.2
- new net: D3.2 (A), R26.1
Changed lines of the file:
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@@
 (kicad_sch (version 20230121) (generator eeschema)
   (paper "A4")
+  (junction (at 104.14 31.75) (diameter 0) (color 0 0 0 0)
+  )
   (junction (at 247.65 27.94) (diameter 0) (color 0 0 0 0)
   )
@@
   )
   (junction (at 238.76 39.37) (diameter 0) (color 0 0 0 0)
+  )
+  (junction (at 73.66 92.71) (diameter 0) (color 0 0 0 0)
   )
   (junction (at 229.87 39.37) (diameter 0) (color 0 0 0 0)
@@
     (stroke (width 0) (type default))
   )
+  (wire (pts (xy 93.98 31.75) (xy 93.98 40.64))
+    (stroke (width 0) (type default))
+  )
   (wire (pts (xy 144.78 35.56) (xy 142.24 35.56))
     (stroke (width 0) (type default))
@@
     (stroke (width 0) (type default))
   )
+  (wire (pts (xy 73.66 92.71) (xy 73.66 95.25))
+    (stroke (width 0) (type default))
+  )
   (wire (pts (xy 154.94 54.61) (xy 162.56 54.61))
     (stroke (width 0) (type default))
@@
     (stroke (width 0) (type default))
   )
+  (wire (pts (xy 114.3 41.91) (xy 124.46 41.91))
+    (stroke (width 0) (type default))
+  )
   (wire (pts (xy 256.54 27.94) (xy 247.65 27.94))
     (stroke (width 0) (type default))
@@
     (stroke (width 0) (type default))
   )
-  (wire (pts (xy 97.79 92.71) (xy 124.46 92.71))
+  (wire (pts (xy 67.31 92.71) (xy 73.66 92.71))
     (stroke (width 0) (type default))
   )
@@
     (stroke (width 0) (type default))
   )
+  (wire (pts (xy 73.66 111.76) (xy 73.66 115.57))
+    (stroke (width 0) (type default))
+  )
   (wire (pts (xy 46.99 179.07) (xy 46.99 182.88))
     (stroke (width 0) (type default))
@@
     (stroke (width 0) (type default))
   )
+  (wire (pts (xy 114.3 31.75) (xy 114.3 41.91))
+    (stroke (width 0) (type default))
+  )
   (wire (pts (xy 48.26 182.88) (xy 48.26 185.42))
     (stroke (width 0) (type default))
@@
     (stroke (width 0) (type default))
   )
+  (wire (pts (xy 73.66 102.87) (xy 73.66 104.14))
+    (stroke (width 0) (type default))
+  )
   (wire (pts (xy 220.98 30.48) (xy 220.98 27.94))
     (stroke (width 0) (type default))
@@
     (stroke (width 0) (type default))
   )
-  (wire (pts (xy 109.22 41.91) (xy 124.46 41.91))
+  (wire (pts (xy 104.14 31.75) (xy 114.3 31.75))
     (stroke (width 0) (type default))
   )
@@
   )
   (wire (pts (xy 247.65 27.94) (xy 238.76 27.94))
+    (stroke (width 0) (type default))
+  )
+  (wire (pts (xy 73.66 92.71) (xy 124.46 92.71))
     (stroke (width 0) (type default))
   )
@@
     (effects (font (size 1.27 1.27)) (justify left bottom))
   )
-  (label "~{RESET}" (at 109.22 41.91 0) (fields_autoplaced)
-    (effects (font (size 1.27 1.27)) (justify left bottom))
-  )
   (label "SWO" (at 113.03 82.55 0) (fields_autoplaced)
     (effects (font (size 1.27 1.27)) (justify left bottom))
@@
     (effects (font (size 1.27 1.27)) (justify left bottom))
   )
+  (label "~{RESET}" (at 106.68 31.75 0) (fields_autoplaced)
+    (effects (font (size 1.27 1.27)) (justify left bottom))
+  )
   (label "SWDIO" (at 171.45 74.93 0) (fields_autoplaced)
     (effects (font (size 1.27 1.27)) (justify left bottom))
@@
     (effects (font (size 1.27 1.27)) (justify left bottom))
   )
-  (hierarchical_label "UART1_RX" (shape input) (at 97.79 92.71 180) (fields_autoplaced)
+  (hierarchical_label "UART1_RX" (shape input) (at 67.31 92.71 180) (fields_autoplaced)
     (effects (font (size 1.27 1.27)) (justify right))
   )
@@
     (effects (font (size 1.27 1.27)) (justify left))
   )
+  (symbol (lib_id "power:GND") (at 93.98 40.64 0) (unit 1)
+    (in_bom yes) (on_board yes) (dnp no) (fields_autoplaced)
+    (property "Reference" "#PWR026" (at 93.98 46.99 0)
+      (effects (font (size 1.27 1.27)) hide)
+    )
+    (property "Value" "GND" (at 93.98 45.72 0)
+      (effects (font (size 1.27 1.27)))
+    )
+    (property "Footprint" "" (at 93.98 40.64 0)
+      (effects (font (size 1.27 1.27)) hide)
+    )
+    (property "Datasheet" "" (at 93.98 40.64 0)
+      (effects (font (size 1.27 1.27)) hide)
+    )
+    (pin "1")
+    (instances
+      (project "minimouse"
+        (path "/d8fa4cba-2469-4231-847f-065b6b829f44/b5d7e952-00af-4b6f-924a-ee43c62726d2"
+          (reference "#PWR026") (unit 1)
+        )
+      )
+    )
+  )
   (symbol (lib_id "Device:R") (at 88.9 52.07 0) (unit 1)
     (in_bom yes) (on_board yes) (dnp no) (fields_autoplaced)
@@
         (path "/d8fa4cba-2469-4231-847f-065b6b829f44/b5d7e952-00af-4b6f-924a-ee43c62726d2"
           (reference "R1") (unit 1)
+        )
+      )
+    )
+  )
+  (symbol (lib_id "Device:R") (at 73.66 99.06 180) (unit 1)
+    (in_bom yes) (on_board yes) (dnp no)
+    (property "Reference" "R26" (at 71.12 99.06 90)
+      (effects (font (size 1.27 1.27)))
+    )
+    (property "Value" "85" (at 72.39 93.98 90)
+      (effects (font (size 1.27 1.27)) hide)
+    )
+    (property "Footprint" "Resistor_SMD:R_0603_1608Metric" (at 75.438 99.06 90)
+      (effects (font (size 1.27 1.27)) hide)
+    )
+    (property "Datasheet" "~" (at 73.66 99.06 0)
+      (effects (font (size 1.27 1.27)) hide)
+    )
+    (pin "1")
+    (pin "2")
+    (instances
+      (project "minimouse"
+        (path "/d8fa4cba-2469-4231-847f-065b6b829f44/b5d7e952-00af-4b6f-924a-ee43c62726d2"
+          (reference "R26") (unit 1)
         )
       )
@@
         (path "/d8fa4cba-2469-4231-847f-065b6b829f44/b5d7e952-00af-4b6f-924a-ee43c62726d2"
           (reference "J1") (unit 1)
+        )
+      )
+    )
+  )
+  (symbol (lib_id "power:GND") (at 73.66 115.57 0) (unit 1)
+    (in_bom yes) (on_board yes) (dnp no) (fields_autoplaced)
+    (property "Reference" "#PWR033" (at 73.66 121.92 0)
+      (effects (font (size 1.27 1.27)) hide)
+    )
+    (property "Value" "GND" (at 73.66 120.65 0)
+      (effects (font (size 1.27 1.27)))
+    )
+    (property "Footprint" "" (at 73.66 115.57 0)
+      (effects (font (size 1.27 1.27)) hide)
+    )
+    (property "Datasheet" "" (at 73.66 115.57 0)
+      (effects (font (size 1.27 1.27)) hide)
+    )
+    (pin "1")
+    (instances
+      (project "minimouse"
+        (path "/d8fa4cba-2469-4231-847f-065b6b829f44/b5d7e952-00af-4b6f-924a-ee43c62726d2"
+          (reference "#PWR033") (unit 1)
         )
       )
@@
     )
   )
+  (symbol (lib_id "power:GND") (at 104.14 39.37 0) (unit 1)
+    (in_bom yes) (on_board yes) (dnp no) (fields_autoplaced)
+    (property "Reference" "#PWR025" (at 104.14 45.72 0)
+      (effects (font (size 1.27 1.27)) hide)
+    )
+    (property "Value" "GND" (at 104.14 44.45 0)
+      (effects (font (size 1.27 1.27)))
+    )
+    (property "Footprint" "" (at 104.14 39.37 0)
+      (effects (font (size 1.27 1.27)) hide)
+    )
+    (property "Datasheet" "" (at 104.14 39.37 0)
+      (effects (font (size 1.27 1.27)) hide)
+    )
+    (pin "1")
+    (instances
+      (project "minimouse"
+        (path "/d8fa4cba-2469-4231-847f-065b6b829f44/b5d7e952-00af-4b6f-924a-ee43c62726d2"
+          (reference "#PWR025") (unit 1)
+        )
+      )
+    )
+  )
+  (symbol (lib_id "Switch:SW_Push") (at 99.06 31.75 0) (unit 1)
+    (in_bom yes) (on_board yes) (dnp no) (fields_autoplaced)
+    (property "Reference" "SW1" (at 99.06 24.13 0)
+      (effects (font (size 1.27 1.27)))
+    )
+    (property "Value" "SW_Push" (at 99.06 26.67 0)
+      (effects (font (size 1.27 1.27)))
+    )
+    (property "Footprint" "Button_Switch_SMD:Panasonic_EVQPUK_EVQPUB" (at 99.06 26.67 0)
+      (effects (font (size 1.27 1.27)) hide)
+    )
+    (property "Datasheet" "~" (at 99.06 26.67 0)
+      (effects (font (size 1.27 1.27)) hide)
+    )
+    (pin "1")
+    (pin "2")
+    (instances
+      (project "minimouse"
+        (path "/d8fa4cba-2469-4231-847f-065b6b829f44/b5d7e952-00af-4b6f-924a-ee43c62726d2"
+          (reference "SW1") (unit 1)
+        )
+      )
+    )
+  )
+  (symbol (lib_id "Device:C") (at 104.14 35.56 0) (unit 1)
+    (in_bom yes) (on_board yes) (dnp no) (fields_autoplaced)
+    (property "Reference" "C16" (at 107.95 34.29 0)
+      (effects (font (size 1.27 1.27)) (justify left))
+    )
+    (property "Value" "100nF" (at 107.95 36.83 0)
+      (effects (font (size 1.27 1.27)) (justify left))
+    )
+    (property "Footprint" "Capacitor_SMD:C_0603_1608Metric" (at 105.1052 39.37 0)
+      (effects (font (size 1.27 1.27)) hide)
+    )
+    (property "Datasheet" "~" (at 104.14 35.56 0)
+      (effects (font (size 1.27 1.27)) hide)
+    )
+    (pin "2")
+    (pin "1")
+    (instances
+      (project "minimouse"
+        (path "/d8fa4cba-2469-4231-847f-065b6b829f44/b5d7e952-00af-4b6f-924a-ee43c62726d2"
+          (reference "C16") (unit 1)
+        )
+      )
+    )
+  )
   (symbol (lib_id "Device:C") (at 238.76 34.29 0) (unit 1)
     (in_bom yes) (on_board yes) (dnp no)
@@
         )
       )
+    )
+  )
+  (symbol (lib_id "Device:LED") (at 73.66 107.95 90) (unit 1)
+    (in_bom yes) (on_board yes) (dnp no) (fields_autoplaced)
+    (property "Reference" "D3" (at 77.47 108.2675 90)
+      (effects (font (size 1.27 1.27)) (justify right))
+    )
+    (property "Value" "red_LED_1.7V_20mA" (at 77.47 110.8075 90)
+      (effects (font (size 1.27 1.27)) (justify right))
+    )
+    (property "Footprint" "LED_SMD:LED_0603_1608Metric" (at 73.66 107.95 0)
+      (effects (font (size 1.27 1.27)) hide)
+    )
+    (property "Datasheet" "~" (at 73.66 107.95 0)
+      (effects (font (size 1.27 1.27)) hide)
+    )
+    (pin "1")
+    (pin "2")
+    (instances
+      (project "minimouse"
+        (path "/d8fa4cba-2469-4231-847f-065b6b829f44/b5d7e952-00af-4b6f-924a-ee43c62726d2"
+          (reference "D3") (unit 1)
+        )
+      )
