File: mm_power.kicad_sch (KiCad schematic)
At the start: 1 part, among them J5 Conn_01x02

Commit message: tp2
Parts:
- added C13: 2.2uF, Capacitor_SMD:C_0603_1608Metric, symbol Device:C
- added C7, C8: 1pF, Capacitor_SMD:C_0603_1608Metric, symbol Device:C
- added D1: red_LED_1.7V_20mA, symbol Device:LED
- added R12: 80, Resistor_SMD:R_0603_1608Metric, symbol Device:R
- added U4: LP5907MFX-3.3, Package_TO_SOT_SMD:SOT-23-5, symbol Regulator_Linear:LP5907MFX-3.3
Connections:
- net +BATT: now also C13.1, C7.1, U4.1 (IN), U4.3 (EN)
- net GND: now also C13.2, C7.2, C8.2, D1.1 (K), U4.2 (GND)
- new net: D1.2 (A), R12.2
- new net +3.3V: C8.1, R12.1, U4.5 (OUT)

Commit message: 31/01
Parts:
- removed C13: 2.2uF, Capacitor_SMD:C_0603_1608Metric, symbol Device:C
- D1: footprint (none) -> LED_SMD:LED_0603_1608Metric
- renumbered C7 to C8, C8 to C9, R12 to R18, U4 to U2
Other:
- moved on the sheet: D1, R18

Commit message: 05/02
Parts:
- added 3.3V1, BATT1, GND1: TestPoint, TestPoint:TestPoint_Pad_D1.5mm, symbol Connector:TestPoint
- added D2: BZT52Bxx, Diode_SMD:D_SOD-123F, symbol Diode:BZT52Bxx
- added Q1: DMP3013SFV, Package_SON:Diodes_PowerDI3333-8, symbol Transistor_FET:DMP3013SFV
- added R24, R25: 10K, Resistor_SMD:R_0603_1608Metric, symbol Device:R
- added R7: 100K, Resistor_SMD:R_0603_1608Metric, symbol Device:R
Connections:
- net +3.3V: now also 3.3V1.1, R25.1
- net +BATT: now also BATT1.1, D2.1 (K), Q1.1 (S), Q1.2 (S), Q1.3 (S), R24.1; no longer J5.2 (Pin_2)
- net GND: now also GND1.1, R24.2, R25.2, R7.2
- new net: D2.2 (A), Q1.4 (G), R7.1
- new net: J5.2 (Pin_2), Q1.5 (D)
Other:
- moved on the sheet: J5
