File: mm_ultrasonic_sensor.kicad_sch (KiCad schematic)
At the start: 0 parts

Commit message: tp2
Parts:
- added C11: 0.1uF, Capacitor_SMD:C_0603_1608Metric, symbol Device:C
- added C12: 2.2uF, Capacitor_SMD:C_0603_1608Metric, symbol Device:C
- added R19: 100, Resistor_SMD:R_0603_1608Metric, symbol Device:R
- added U2: HC-SR04, minimouse:HC-SR04, symbol minimouse:HC-SR04
Connections:
- net SONAR_ECHO: now also R19.1
- net SONAR_TRIGGER: now also U2.2 (TRIG)
- new net: R19.2, U2.3 (ECHO)
- new net +BATT: C11.1, C12.1, U2.4 (VCC)
- new net GND: C11.2, C12.2, U2.1 (GND)

Commit message: 31/01
Parts:
- removed C11: 0.1uF, Capacitor_SMD:C_0603_1608Metric, symbol Device:C
- renumbered C12 to C15, R19 to R23, U2 to U4
Connections:
- net +BATT renamed +3.3V
Other:
- moved on the sheet: C15
Changed lines of the file:
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@@
 (kicad_sch (version 20230121) (generator eeschema)
   (paper "A4")
-  (junction (at 133.35 48.26) (diameter 0) (color 0 0 0 0)
-  )
-  (junction (at 133.35 59.69) (diameter 0) (color 0 0 0 0)
-  )
-  (wire (pts (xy 88.9 73.66) (xy 92.71 73.66))
-    (stroke (width 0) (type default))
-  )
-  (wire (pts (xy 88.9 72.39) (xy 88.9 73.66))
+  (wire (pts (xy 72.39 73.66) (xy 92.71 73.66))
     (stroke (width 0) (type default))
   )
@@
     (stroke (width 0) (type default))
   )
-  (wire (pts (xy 138.43 48.26) (xy 138.43 49.53))
-    (stroke (width 0) (type default))
-  )
-  (wire (pts (xy 127 48.26) (xy 133.35 48.26))
-    (stroke (width 0) (type default))
-  )
-  (wire (pts (xy 138.43 57.15) (xy 138.43 59.69))
-    (stroke (width 0) (type default))
-  )
   (wire (pts (xy 102.87 85.09) (xy 102.87 88.9))
-    (stroke (width 0) (type default))
-  )
-  (wire (pts (xy 138.43 48.26) (xy 133.35 48.26))
     (stroke (width 0) (type default))
   )
@@
     (stroke (width 0) (type default))
   )
-  (wire (pts (xy 87.63 72.39) (xy 88.9 72.39))
-    (stroke (width 0) (type default))
-  )
-  (wire (pts (xy 127 48.26) (xy 127 49.53))
-    (stroke (width 0) (type default))
-  )
-  (wire (pts (xy 127 59.69) (xy 133.35 59.69))
-    (stroke (width 0) (type default))
-  )
-  (wire (pts (xy 138.43 59.69) (xy 133.35 59.69))
-    (stroke (width 0) (type default))
-  )
   (wire (pts (xy 102.87 64.77) (xy 102.87 57.15))
     (stroke (width 0) (type default))
   )
-  (wire (pts (xy 127 57.15) (xy 127 59.69))
+  (wire (pts (xy 133.35 57.15) (xy 133.35 59.69))
     (stroke (width 0) (type default))
   )
-  (wire (pts (xy 133.35 48.26) (xy 133.35 46.99))
+  (wire (pts (xy 133.35 46.99) (xy 133.35 49.53))
     (stroke (width 0) (type default))
   )
-  (hierarchical_label "SONAR_TRIGGER" (shape input) (at 87.63 72.39 180) (fields_autoplaced)
+  (hierarchical_label "SONAR_TRIGGER" (shape input) (at 72.39 73.66 180) (fields_autoplaced)
     (effects (font (size 1.27 1.27)) (justify right))
   )
@@
   (symbol (lib_id "Device:R") (at 82.55 76.2 90) (unit 1)
     (in_bom yes) (on_board yes) (dnp no)
-    (property "Reference" "R19" (at 76.2 74.93 90)
+    (property "Reference" "R23" (at 76.2 74.93 90)
       (effects (font (size 1.27 1.27)))
     )
@@
       (project "minimouse"
         (path "/d8fa4cba-2469-4231-847f-065b6b829f44/224298a9-7d6e-4a70-a0a5-f2614895ec28"
-          (reference "R19") (unit 1)
-        )
-      )
-    )
-  )
-  (symbol (lib_id "Device:C") (at 138.43 53.34 0) (unit 1)
-    (in_bom yes) (on_board yes) (dnp no) (fields_autoplaced)
-    (property "Reference" "C11" (at 142.24 52.07 0)
-      (effects (font (size 1.27 1.27)) (justify left))
-    )
-    (property "Value" "0.1uF" (at 142.24 54.61 0)
-      (effects (font (size 1.27 1.27)) (justify left))
-    )
-    (property "Footprint" "Capacitor_SMD:C_0603_1608Metric" (at 139.3952 57.15 0)
-      (effects (font (size 1.27 1.27)) hide)
-    )
-    (property "Datasheet" "~" (at 138.43 53.34 0)
-      (effects (font (size 1.27 1.27)) hide)
-    )
-    (pin "1")
-    (pin "2")
-    (instances
-      (project "minimouse"
-        (path "/d8fa4cba-2469-4231-847f-065b6b829f44/224298a9-7d6e-4a70-a0a5-f2614895ec28"
-          (reference "C11") (unit 1)
+          (reference "R23") (unit 1)
         )
       )
@@
   (symbol (lib_id "minimouse:HC-SR04") (at 102.87 74.93 0) (unit 1)
     (in_bom yes) (on_board yes) (dnp no) (fields_autoplaced)
-    (property "Reference" "U2" (at 115.57 73.66 0)
+    (property "Reference" "U4" (at 115.57 73.66 0)
       (effects (font (size 1.27 1.27)) (justify left))
     )
@@
       (project "minimouse"
         (path "/d8fa4cba-2469-4231-847f-065b6b829f44/224298a9-7d6e-4a70-a0a5-f2614895ec28"
-          (reference "U2") (unit 1)
+          (reference "U4") (unit 1)
         )
       )
     )
   )
-  (symbol (lib_id "power:+BATT") (at 102.87 57.15 0) (unit 1)
+  (symbol (lib_id "power:+3.3V") (at 133.35 46.99 0) (unit 1)
     (in_bom yes) (on_board yes) (dnp no) (fields_autoplaced)
-    (property "Reference" "#PWR025" (at 102.87 60.96 0)
+    (property "Reference" "#PWR010" (at 133.35 50.8 0)
       (effects (font (size 1.27 1.27)) hide)
     )
-    (property "Value" "+BATT" (at 102.87 52.07 0)
+    (property "Value" "+3.3V" (at 133.35 41.91 0)
+      (effects (font (size 1.27 1.27)))
+    )
+    (property "Footprint" "" (at 133.35 46.99 0)
+      (effects (font (size 1.27 1.27)) hide)
+    )
+    (property "Datasheet" "" (at 133.35 46.99 0)
+      (effects (font (size 1.27 1.27)) hide)
+    )
+    (pin "1")
+    (instances
+      (project "minimouse"
+        (path "/d8fa4cba-2469-4231-847f-065b6b829f44/224298a9-7d6e-4a70-a0a5-f2614895ec28"
+          (reference "#PWR010") (unit 1)
+        )
+      )
+    )
+  )
+  (symbol (lib_id "power:+3.3V") (at 102.87 57.15 0) (unit 1)
+    (in_bom yes) (on_board yes) (dnp no) (fields_autoplaced)
+    (property "Reference" "#PWR012" (at 102.87 60.96 0)
+      (effects (font (size 1.27 1.27)) hide)
+    )
+    (property "Value" "+3.3V" (at 102.87 52.07 0)
       (effects (font (size 1.27 1.27)))
     )
@@
       (project "minimouse"
         (path "/d8fa4cba-2469-4231-847f-065b6b829f44/224298a9-7d6e-4a70-a0a5-f2614895ec28"
-          (reference "#PWR025") (unit 1)
+          (reference "#PWR012") (unit 1)
         )
       )
     )
   )
-  (symbol (lib_id "power:+BATT") (at 133.35 46.99 0) (unit 1)
-    (in_bom yes) (on_board yes) (dnp no) (fields_autoplaced)
-    (property "Reference" "#PWR026" (at 133.35 50.8 0)
+  (symbol (lib_id "Device:C") (at 133.35 53.34 0) (unit 1)
+    (in_bom yes) (on_board yes) (dnp no)
+    (property "Reference" "C15" (at 125.73 52.07 0)
+      (effects (font (size 1.27 1.27)) (justify left))
+    )
+    (property "Value" "2.2uF" (at 125.73 55.88 0)
+      (effects (font (size 1.27 1.27)) (justify left))
+    )
+    (property "Footprint" "Capacitor_SMD:C_0603_1608Metric" (at 134.3152 57.15 0)
       (effects (font (size 1.27 1.27)) hide)
     )
-    (property "Value" "+BATT" (at 133.35 41.91 0)
-      (effects (font (size 1.27 1.27)))
-    )
-    (property "Footprint" "" (at 133.35 46.99 0)
-      (effects (font (size 1.27 1.27)) hide)
-    )
-    (property "Datasheet" "" (at 133.35 46.99 0)
-      (effects (font (size 1.27 1.27)) hide)
-    )
-    (pin "1")
-    (instances
-      (project "minimouse"
-        (path "/d8fa4cba-2469-4231-847f-065b6b829f44/224298a9-7d6e-4a70-a0a5-f2614895ec28"
-          (reference "#PWR026") (unit 1)
-        )
-      )
-    )
-  )
-  (symbol (lib_id "Device:C") (at 127 53.34 0) (unit 1)
-    (in_bom yes) (on_board yes) (dnp no)
-    (property "Reference" "C12" (at 119.38 52.07 0)
-      (effects (font (size 1.27 1.27)) (justify left))
-    )
-    (property "Value" "2.2uF" (at 119.38 55.88 0)
-      (effects (font (size 1.27 1.27)) (justify left))
-    )
-    (property "Footprint" "Capacitor_SMD:C_0603_1608Metric" (at 127.9652 57.15 0)
-      (effects (font (size 1.27 1.27)) hide)
-    )
-    (property "Datasheet" "~" (at 127 53.34 0)
+    (property "Datasheet" "~" (at 133.35 53.34 0)
       (effects (font (size 1.27 1.27)) hide)
     )
@@
       (project "minimouse"
         (path "/d8fa4cba-2469-4231-847f-065b6b829f44/224298a9-7d6e-4a70-a0a5-f2614895ec28"
-          (reference "C12") (unit 1)
+          (reference "C15") (unit 1)
         )
       )

Commit message: 05/02
Connections:
- net +3.3V renamed +BATT
Changed lines of the file:
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@@
     )
   )
-  (symbol (lib_id "power:+3.3V") (at 133.35 46.99 0) (unit 1)
+  (symbol (lib_id "power:+BATT") (at 102.87 57.15 0) (unit 1)
+    (in_bom yes) (on_board yes) (dnp no) (fields_autoplaced)
+    (property "Reference" "#PWR012" (at 102.87 60.96 0)
+      (effects (font (size 1.27 1.27)) hide)
+    )
+    (property "Value" "+BATT" (at 102.87 52.07 0)
+      (effects (font (size 1.27 1.27)))
+    )
+    (property "Footprint" "" (at 102.87 57.15 0)
+      (effects (font (size 1.27 1.27)) hide)
+    )
+    (property "Datasheet" "" (at 102.87 57.15 0)
+      (effects (font (size 1.27 1.27)) hide)
+    )
+    (pin "1")
+    (instances
+      (project "minimouse"
+        (path "/d8fa4cba-2469-4231-847f-065b6b829f44/224298a9-7d6e-4a70-a0a5-f2614895ec28"
+          (reference "#PWR012") (unit 1)
+        )
+      )
+    )
+  )
+  (symbol (lib_id "power:+BATT") (at 133.35 46.99 0) (unit 1)
     (in_bom yes) (on_board yes) (dnp no) (fields_autoplaced)
     (property "Reference" "#PWR010" (at 133.35 50.8 0)
       (effects (font (size 1.27 1.27)) hide)
     )
-    (property "Value" "+3.3V" (at 133.35 41.91 0)
+    (property "Value" "+BATT" (at 133.35 41.91 0)
       (effects (font (size 1.27 1.27)))
     )
@@
         )
       )
-    )
-  )
-  (symbol (lib_id "power:+3.3V") (at 102.87 57.15 0) (unit 1)
-    (in_bom yes) (on_board yes) (dnp no) (fields_autoplaced)
-    (property "Reference" "#PWR012" (at 102.87 60.96 0)
-      (effects (font (size 1.27 1.27)) hide)
-    )
-    (property "Value" "+3.3V" (at 102.87 52.07 0)
-      (effects (font (size 1.27 1.27)))
-    )
-    (property "Footprint" "" (at 102.87 57.15 0)
-      (effects (font (size 1.27 1.27)) hide)
-    )
-    (property "Datasheet" "" (at 102.87 57.15 0)
-      (effects (font (size 1.27 1.27)) hide)
-    )
-    (pin "1")
-    (instances
-      (project "minimouse"
-        (path "/d8fa4cba-2469-4231-847f-065b6b829f44/224298a9-7d6e-4a70-a0a5-f2614895ec28"
-          (reference "#PWR012") (unit 1)
-        )
-      )
